Commit message: Driving the robot in Gazebo and visualizing in Rviz

File: ros2_ws/src/amr_description/urdf/robot.urdf.xacro (robot description, xacro)
@@ -2,3 +2,4 @@
 <robot xmlns:xacro="http://www.ros.org/wiki/xacro"  name="robot">
     <xacro:include filename="robot_core.xacro" />
+    <xacro:include filename="gazebo_control.xacro"/>
 </robot>

File: ros2_ws/src/amr_description/urdf/robot_core.xacro (robot description, xacro)
@@ -109,3 +109,16 @@
         </xacro:inertial_sphere>
     </link>
+    <!-- GAZEBO MATERIALS -->
+    <gazebo reference="chassis">
+    <material>Gazebo/White</material>
+    </gazebo>
+    <gazebo reference="left_wheel">
+    <material>Gazebo/Blue</material>
+    </gazebo>
+    <gazebo reference="right_wheel">
+    <material>Gazebo/Blue</material>
+    </gazebo>
+    <gazebo reference="caster_wheel">
+    <material>Gazebo/Black</material>
+    </gazebo>
 </robot>
