Commit message: Feat : add launch and parameters for the real robot

File: ros2_ws/src/amr_control/urdf/ros2_control.xacro (robot description, xacro)
@@ -2,27 +2,64 @@
 <robot xmlns:xacro="http://www.ros.org/wiki/xacro">
   <xacro:macro name="ros2_control" params="name initial_positions_file:=''">
-    <ros2_control name="${name}" type="system">
-      <hardware>
-        <plugin>gz_ros2_control/GazeboSimSystem</plugin>
-      </hardware>
-      <!-- Left wheel -->
-      <joint name="left_wheel_joint">
-        <command_interface name="velocity">
-          <param name="min">-10.0</param>
-          <param name="max">10.0</param>
-        </command_interface>
-        <state_interface name="position"/>
-        <state_interface name="velocity"/>
-      </joint>
-      <!-- Right wheel -->
-      <joint name="right_wheel_joint">
-        <command_interface name="velocity">
-          <param name="min">-10.0</param>
-          <param name="max">10.0</param>
-        </command_interface>
-        <state_interface name="position"/>
-        <state_interface name="velocity"/>
-      </joint>
-    </ros2_control>
+    <xacro:unless value="$(arg sim_mode)">
+      <ros2_control name="RealRobot" type="system">
+        <hardware>
+          <plugin>diffdrive_arduino/DiffDriveArduinoHardware</plugin>
+          <param name="left_wheel_name">left_wheel_joint</param>
+          <param name="right_wheel_name">right_wheel_joint</param>
+          <param name="loop_rate">30</param>
+          <param name="device">/dev/ttyACM0</param>
+          <param name="baud_rate">57600</param>
+          <param name="timeout_ms">1000</param>
+          <param name="left_enc_counts_per_rev">441</param>
+          <param name="right_enc_counts_per_rev">441</param>
+          <param name="pid_p">20</param>
+          <param name="pid_d">12</param>
+          <param name="pid_i">0</param>
+          <param name="pid_o">50</param>
+        </hardware>
+        <joint name="left_wheel_joint">
+          <command_interface name="velocity">
+            <param name="min">-10</param>
+            <param name="max">10</param>
+          </command_interface>
+          <state_interface name="position"/>
+          <state_interface name="velocity"/>
+        </joint>
+        <joint name="right_wheel_joint">
+          <command_interface name="velocity">
+            <param name="min">-10</param>
+            <param name="max">10</param>
+          </command_interface>
+          <state_interface name="position"/>
+          <state_interface name="velocity"/>
+        </joint>
+      </ros2_control>
+    </xacro:unless>
+    <xacro:if value="$(arg sim_mode)">
+      <ros2_control name="${name}" type="system">
+        <hardware>
+          <plugin>gz_ros2_control/GazeboSimSystem</plugin>
+        </hardware>
+        <!-- Left wheel -->
+        <joint name="left_wheel_joint">
+          <command_interface name="velocity">
+            <param name="min">-10.0</param>
+            <param name="max">10.0</param>
+          </command_interface>
+          <state_interface name="position"/>
+          <state_interface name="velocity"/>
+        </joint>
+        <!-- Right wheel -->
+        <joint name="right_wheel_joint">
+          <command_interface name="velocity">
+            <param name="min">-10.0</param>
+            <param name="max">10.0</param>
+          </command_interface>
+          <state_interface name="position"/>
+          <state_interface name="velocity"/>
+        </joint>
+      </ros2_control>
+    </xacro:if>
     <gazebo>
         <plugin

File: ros2_ws/src/amr_description/urdf/robot.urdf.xacro (robot description, xacro)
@@ -1,9 +1,15 @@
 <?xml version="1.0"?>
 <robot xmlns:xacro="http://www.ros.org/wiki/xacro"  name="robot">
+    <xacro:arg name="use_ros2_control" default="true"/>
+    <xacro:arg name="sim_mode" default="false"/>
     <xacro:include filename="robot_core.xacro"/>
-    <xacro:include filename="$(find amr_simulation)/urdf/gazebo.xacro"/>
     <xacro:include filename="lidar.xacro"/>
-    <xacro:include filename="$(find amr_control)/urdf/ros2_control.xacro"/>
-    <xacro:ros2_control name="GazeboSimSystem"/>
+    <xacro:if value="$(arg use_ros2_control)">
+        <xacro:include filename="$(find amr_control)/urdf/ros2_control.xacro"/>
+        <xacro:ros2_control name="AMRSystem"/>
+    </xacro:if>
+    <xacro:unless value="$(arg use_ros2_control)">
+        <xacro:include filename="$(find amr_simulation)/urdf/gazebo.xacro"/>
+    </xacro:unless>
     <xacro:include filename="camera.xacro"/>
     <xacro:arg name="show_camera_fov" default="false"/>

Commit message: Fix : correct the simulation launch and changed the joysticks params

File: ros2_ws/src/amr_control/urdf/ros2_control.xacro (robot description, xacro)
@@ -1,5 +1,7 @@
 <?xml version="1.0"?>
 <robot xmlns:xacro="http://www.ros.org/wiki/xacro">
-  <xacro:macro name="ros2_control" params="name initial_positions_file:=''">
+  <xacro:macro
+      name="ros2_control"
+      params="name initial_positions_file:='' controller_params_file">
     <xacro:unless value="$(arg sim_mode)">
       <ros2_control name="RealRobot" type="system">
@@ -62,11 +64,13 @@
       </ros2_control>
     </xacro:if>
-    <gazebo>
-        <plugin
-            filename="libgz_ros2_control-system.so"
-            name="gz_ros2_control::GazeboSimROS2ControlPlugin">
-            <parameters>$(find amr_control)/config/controllers.yaml</parameters>
-        </plugin>
-    </gazebo>
+    <xacro:if value="$(arg sim_mode)">
+      <gazebo>
+          <plugin
+              filename="libgz_ros2_control-system.so"
+              name="gz_ros2_control::GazeboSimROS2ControlPlugin">
+              <parameters>${controller_params_file}</parameters>
+          </plugin>
+      </gazebo>
+    </xacro:if>
     <gazebo reference="left_wheel">
         <mu1>1.0</mu1>

File: ros2_ws/src/amr_description/urdf/robot.urdf.xacro (robot description, xacro)
@@ -3,9 +3,16 @@
     <xacro:arg name="use_ros2_control" default="true"/>
     <xacro:arg name="sim_mode" default="false"/>
+    <xacro:arg
+        name="controller_params_file"
+        default="$(find amr_control)/config/controllers.yaml"
+    />
     <xacro:include filename="robot_core.xacro"/>
     <xacro:include filename="lidar.xacro"/>
     <xacro:if value="$(arg use_ros2_control)">
         <xacro:include filename="$(find amr_control)/urdf/ros2_control.xacro"/>
-        <xacro:ros2_control name="AMRSystem"/>
+        <xacro:ros2_control
+            name="AMRSystem"
+            controller_params_file="$(arg controller_params_file)"
+        />
     </xacro:if>
     <xacro:unless value="$(arg use_ros2_control)">
@@ -13,4 +20,3 @@
     </xacro:unless>
     <xacro:include filename="camera.xacro"/>
-    <xacro:arg name="show_camera_fov" default="false"/>
 </robot>
